File: schematics/circuit-new.brd (EAGLE design)
At the start: 100 x 80 mm, 66 parts, among them IC1 TLC271D, IC2 TLC271D, U1 AD5241BRU1M-REEL7AD5241BRZ1M, X2 87758-0216, X3 87758-0216, X4 87758-0216, X5 87758-0216, X8 87758-0216, X9 87758-0216

Commit message: Последняя версия платы и схемы
Parts:
- added E$1: (no value), SparkFun-Resistors:0805
- added R10: 10, SparkFun-Resistors:0402-RES
Changed lines of the file:
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@@
 <setting verticaltext="up"/>
 </settings>
-<grid distance="0.1" unitdist="mm" unit="mm" style="lines" multiple="1" display="yes" altdistance="1" altunitdist="mm" altunit="mm"/>
+<grid distance="1" unitdist="mm" unit="mm" style="lines" multiple="1" display="yes" altdistance="1" altunitdist="mm" altunit="mm"/>
 <layers>
 <layer number="1" name="Top" color="4" fill="1" visible="yes" active="yes"/>
@@
 <element name="U2" library="elements" package="SOT223" value="" x="55.5" y="18.6" rot="R270"/>
 <element name="U3" library="elements" package="SOT223" value="" x="44.1" y="18.8" rot="R90"/>
+<element name="R10" library="SparkFun-Resistors" package="0402-RES" value="10" x="1.27" y="0.74"/>
+<element name="E$1" library="SparkFun-Resistors" package="0805" value="" x="22" y="14"/>
 </elements>
 <signals>
