File: schematics/circuit-main.brd (EAGLE design)
At the start: 100 x 80 mm, 54 parts, among them IC1 TLC271D, IC2 TLC271D, U1 AD5241BRU1M-REEL7AD5241BRZ1M, X1 87758-0216, X10 87758-0216, X2 87758-0216, X3 87758-0216, X4 87758-0216, X6 87758-0216, X7 87758-0216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

Commit message: готовые 2 платы
Parts:
- removed HMDT: (no value), RHT03_DHT-22_AM2302:RHT03_DHT-22/RA
- removed R13, R14: 0.75, SparkFun-Resistors:0805
- removed X10, X8: 87758-0216, con-molex:87758-0216
- added R2, R3: 0.75, SparkFun-Resistors:0805
- added U4: (no value), RHT03_DHT-22_AM2302:RHT03_DHT-22/RA
- added X5: 87758-0216, con-molex:87758-0216
- moved PROBE_8 12.0 mm to (51.6, 57.5)
- moved X3 6.29 mm to (55.2, 52.9), turned to 90 degrees
- moved Q4 5.89 mm to (55.2, 57.5), turned to 270 degrees
- moved Q7 4.75 mm to (45.7, 34.4)
- moved IC1 4.53 mm to (39.7, 45.1)
- moved R1 4.14 mm to (48.3, 26.2), turned to 0 degrees
- moved GROUND_PROBE1 3.03 mm to (73.5, 24.4)
- moved R25 2.94 mm to (49.2, 43.5), turned to 270 degrees
- moved IC2 2.51 mm to (44.2, 57.1)
- moved X6 1.33 mm to (65.4, 36.0)
- moved R12 1.15 mm to (79.7, 36.0)
- moved U1 0.83 mm to (61.1, 45.8)
- moved X7 0.73 mm to (20.8, 42.1)
- moved U$3 0.53 mm to (25.8, 37.1)
- moved R26 0.38 mm to (80.3, 41.3)
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Connections:
- removed net N$10: IC2.2, R13.1, R14.2
- removed net N$55: HMDT.DATA, R1.1, X8.1
- removed net V+: IC1.7, IC2.7
- removed net VCC: IC2.1
- new net N$1: IC2.6, R2.1, X5.1
- new net N$110: IC2.3, R12.2, U$4.VOUT
- new net N$111: IC1.2, R25.1, R26.2
- new net N$3: R1.2, U4.DATA, X5.2
- net 3.3V: now also R1.1, U4.VDD; no longer HMDT.VDD, R1.2
- net 5V: now also IC1.7, IC1.8, IC2.7, IC2.8; no longer IC1.1, IC1.2, IC2.3, R12.2, R25.1, R26.2, U$4.VOUT
- net GND: now also R3.2, U4.GND; no longer HMDT.GND, R14.1
- net N$4: now also IC2.2, R2.2, R3.1; no longer IC2.6, R13.2, X10.1
Routing:
- net N$110: track 0.00 -> 127.6 mm, vias 0 -> 5
- net N$111: track 0.00 -> 110.8 mm, vias 0 -> 4
- net 5V: track 269.9 -> 209.9 mm, vias 17 -> 13
- net N$1: track 0.00 -> 34.1 mm, vias 0 -> 1
- net N$9: track 193.5 -> 159.4 mm
- net N$55: track 33.9 -> 0.00 mm, vias 3 -> 0
- net N$3: track 0.00 -> 27.0 mm, vias 0 -> 1
- net V+: track 25.4 -> 0.00 mm, vias 1 -> 0
- net N$19: track 66.2 -> 44.3 mm, vias 2 -> 0
- net GND: track 315.9 -> 330.0 mm, vias 12 -> 15
- net N$24: track 14.4 -> 28.4 mm, vias 0 -> 2
- net N$4: track 28.1 -> 14.6 mm, vias 2 -> 0
- net N$10: track 11.9 -> 0.00 mm
- net N$22: track 70.3 -> 78.5 mm
- net SCL_5V: track 33.5 -> 37.5 mm
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