File: schematics/circuit-main.sch (EAGLE design)
At the start: 54 parts, among them IC1 TLC271D, IC2 TLC271D, U1 AD5241BRU1M-REEL7AD5241BRZ1M, X1 87758-0216, X10 87758-0216, X2 87758-0216, X3 87758-0216, X4 87758-0216, X6 87758-0216, X7 87758-0216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

Commit message: готовые 2 платы
Parts:
- removed HMDT: (no value), RHT03_DHT-22_AM2302:RHT03_DHT-22_AM2302RA
- removed R13, R14: 0.75, SparkFun-Resistors:0.75OHM-1/4W-1%(0805)
- removed X10, X8: 87758-0216, con-molex:87758-0216
- added R2, R3: 0.75, SparkFun-Resistors:0.75OHM-1/4W-1%(0805)
- added U4: (no value), RHT03_DHT-22_AM2302:RHT03_DHT-22_AM2302RA
- added X5: 87758-0216, con-molex:87758-0216
Connections:
- removed net N$10: IC2.-IN, R13.1, R14.2
- removed net N$55: HMDT.DATA, R1.1, X8-1.S
- removed net VCC: IC2.ON1
- new net N$1: IC2.OUT, R2.1, X5-1.S
- new net N$110: IC2.+IN, R12.2, U$4.VOUT
- new net N$111: IC1.-IN, R25.1, R26.2
- new net N$3: R1.2, U4.DATA, X5-2.S
- net 3.3V: now also R1.1, U4.VDD; no longer HMDT.VDD, R1.2
- net 5V: now also IC1.OPT, IC1.V+, IC2.OPT, IC2.V+; no longer IC1.-IN, IC1.ON1, IC2.+IN, R12.2, R25.1, R26.2, U$4.VOUT
- net GND: now also R3.2, U4.GND; no longer HMDT.GND, R14.1
- net N$4: now also IC2.-IN, R2.2, R3.1; no longer IC2.OUT, R13.2, X10-1.S
Other:
- moved on the sheet: IC2, R1, R12, R20, R21, U$4, X2-1, X2-2
