File: schematics/smallcircuit.brd (EAGLE design)
At the start: 100 x 80 mm, 8 parts, among them U1 ADXL375BCCZ, X3 87758-0616

Commit message: готовые 2 платы
Parts:
- removed X3: 87758-0616, con-molex:87758-0616
- added X1: 87758-0816, con-molex:87758-0816
- moved R2 17.5 mm to (44.8, 47.6)
- moved R1 12.7 mm to (49.0, 48.9), turned to 90 degrees
- moved U$1 9.38 mm to (46.2, 36.1), turned to 90 degrees
- moved U1 8.62 mm to (56.0, 38.5), turned to 90 degrees
- moved R3 6.74 mm to (44.1, 43.7)
- moved C2 5.73 mm to (40.9, 39.7)
- moved C1 0.28 mm to (54.5, 34.2), turned to 0 degrees
Connections:
- removed net SCL_3.3V: R1.2, R2.2, U$1.5, U$1.6, U1.13, U1.14
- new net N$2: R2.2, U$1.6, U1.13
- new net N$5: R1.2, U$1.5, U1.14
- new net N$7: R2.1, X1.2
- new net N$8: U1.9, X1.8
- net 3.3V: now also X1.5; no longer X3.5
- net GND: now also U$1.PLANE, X1.3; no longer X3.3
- net N$1: now also X1.1; no longer X3.1
- net N$3: now also U1.8, X1.6; no longer R1.1, X3.6
- net N$4: now also R1.1, X1.4; no longer R2.1, X3.4
Routing:
- net N$5: track 0.00 -> 43.7 mm, vias 0 -> 3
- net SCL_3.3V: track 41.1 -> 0.00 mm, vias 2 -> 0
- net GND: track 77.7 -> 52.3 mm, vias 2 -> 3
- net N$2: track 0.00 -> 25.2 mm, vias 0 -> 2
- net N$3: track 6.23 -> 17.0 mm
- net N$8: track 0.00 -> 10.3 mm
- net N$7: track 0.00 -> 4.73 mm
- net N$4: track 6.14 -> 1.99 mm
- net N$6: track 12.2 -> 8.40 mm, vias 2 -> 0
- net N$1: track 15.9 -> 19.0 mm, vias 2 -> 0
- net 3.3V: track 86.3 -> 87.4 mm, vias 6 -> 0
