File: schematics/smallcircuit.sch (EAGLE design)
At the start: 8 parts, among them U1 ADXL375BCCZ, X3 87758-0616

Commit message: готовые 2 платы
Parts:
- removed X3: 87758-0616, con-molex:87758-0616
- added X1: 87758-0816, con-molex:87758-0816
Connections:
- removed net SCL_3.3V: R1.2, R2.2, U$1.SCL, U$1.SDA, U1.SCL/SCLK, U1.SDA/SDI/SDIO
- new net N$2: R2.2, U$1.SDA, U1.SDA/SDI/SDIO
- new net N$5: R1.2, U$1.SCL, U1.SCL/SCLK
- new net N$7: R2.1, X1-2.S
- new net N$8: U1.INT2, X1-8.S
- net 3.3V: now also X1-5.S; no longer X3-5.S
- net GND: now also U$1.PLANE, X1-3.S; no longer X3-3.S
- net N$1: now also X1-1.S; no longer X3-1.S
- net N$3: now also U1.INT1, X1-6.S; no longer R1.1, X3-6.S
- net N$4: now also R1.1, X1-4.S; no longer R2.1, X3-4.S
Other:
- moved on the sheet: R3
Changed lines of the file:
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@@
 <part name="C2" library="SparkFun-Passives" deviceset="CAP_POL" device="3528"/>
 <part name="GND3" library="SparkFun-Aesthetics" deviceset="GND" device=""/>
-<part name="X3" library="con-molex" deviceset="87758-0616" device=""/>
+<part name="GND4" library="SparkFun-Aesthetics" deviceset="GND" device=""/>
+<part name="X1" library="con-molex" deviceset="87758-0816" device=""/>
 </parts>
 <sheets>
@@
 <instances>
 <instance part="GND1" gate="1" x="-22.92" y="-10.5"/>
-<instance part="R3" gate="G$1" x="22.86" y="-10.16"/>
+<instance part="R3" gate="G$1" x="22.86" y="-5.08"/>
 <instance part="U1" gate="A" x="104.14" y="7.62"/>
 <instance part="GND2" gate="1" x="142.24" y="5.08"/>
@@
 <instance part="C2" gate="G$1" x="35.56" y="38.1"/>
 <instance part="GND3" gate="1" x="35.56" y="22.86"/>
-<instance part="X3" gate="-1" x="-27.94" y="5.08" rot="R90"/>
-<instance part="X3" gate="-2" x="165.1" y="40.64"/>
-<instance part="X3" gate="-3" x="27.94" y="22.86" rot="R270"/>
-<instance part="X3" gate="-4" x="50.8" y="-17.78" rot="R270"/>
-<instance part="X3" gate="-5" x="45.72" y="53.34" rot="R90"/>
-<instance part="X3" gate="-6" x="40.64" y="-20.32" rot="R270"/>
+<instance part="GND4" gate="1" x="10.16" y="-20.32"/>
+<instance part="X1" gate="-1" x="-27.94" y="5.08" rot="R90"/>
+<instance part="X1" gate="-2" x="50.8" y="-20.32" rot="R270"/>
+<instance part="X1" gate="-3" x="27.94" y="22.86" rot="R270"/>
+<instance part="X1" gate="-4" x="40.64" y="-20.32" rot="R270"/>
+<instance part="X1" gate="-5" x="45.72" y="53.34" rot="R90"/>
+<instance part="X1" gate="-6" x="142.24" y="20.32"/>
+<instance part="X1" gate="-7" x="101.6" y="53.34"/>
+<instance part="X1" gate="-8" x="142.24" y="17.78"/>
 </instances>
 <busses>
@@
 <segment>
 <pinref part="R3" gate="G$1" pin="2"/>
-<wire x1="27.94" y1="-10.16" x2="30.48" y2="-10.16" width="0.1524" layer="91"/>
-<wire x1="30.48" y1="-10.16" x2="30.48" y2="15.24" width="0.1524" layer="91"/>
+<wire x1="27.94" y1="-5.08" x2="30.48" y2="-5.08" width="0.1524" layer="91"/>
+<wire x1="30.48" y1="-5.08" x2="30.48" y2="15.24" width="0.1524" layer="91"/>
 <pinref part="U1" gate="A" pin="*CS"/>
 <wire x1="76.2" y1="-5.08" x2="71.12" y2="-5.08" width="0.1524" layer="91"/>
@@
 <wire x1="35.56" y1="40.64" x2="35.56" y2="43.18" width="0.1524" layer="91"/>
 <junction x="35.56" y="43.18"/>
-<pinref part="X3" gate="-5" pin="S"/>
+<pinref part="X1" gate="-5" pin="S"/>
 </segment>
 </net>
@@
 <junction x="27.94" y="27.94"/>
 <pinref part="GND3" gate="1" pin="GND"/>
-<pinref part="X3" gate="-3" pin="S"/>
+<pinref part="X1" gate="-3" pin="S"/>
+</segment>
+<segment>
+<pinref part="U$1" gate="G$1" pin="PLANE"/>
+<wire x1="5.08" y1="-10.16" x2="10.16" y2="-10.16" width="0.1524" layer="91"/>
+<wire x1="10.16" y1="-10.16" x2="10.16" y2="-17.78" width="0.1524" layer="91"/>
+<pinref part="GND4" gate="1" pin="GND"/>
 </segment>
 </net>
@@
 <wire x1="-27.94" y1="0" x2="-27.94" y2="2.54" width="0.1524" layer="91"/>
 <pinref part="U$1" gate="G$1" pin="ADDR"/>
-<pinref part="X3" gate="-1" pin="S"/>
+<pinref part="X1" gate="-1" pin="S"/>
 </segment>
 </net>
 <net name="N$6" class="0">
 <segment>
-<wire x1="15.24" y1="-5.08" x2="15.24" y2="-10.16" width="0.1524" layer="91"/>
 <pinref part="R3" gate="G$1" pin="1"/>
-<wire x1="15.24" y1="-10.16" x2="17.78" y2="-10.16" width="0.1524" layer="91"/>
+<wire x1="15.24" y1="-5.08" x2="17.78" y2="-5.08" width="0.1524" layer="91"/>
 <pinref part="U$1" gate="G$1" pin="INT"/>
 </segment>
 </net>
-<net name="SCL_3.3V" class="0">
-<segment>
-<wire x1="15.24" y1="5.08" x2="50.8" y2="5.08" width="0.1524" layer="91"/>
-<pinref part="R2" gate="G$1" pin="2"/>
-<wire x1="50.8" y1="-2.54" x2="50.8" y2="5.08" width="0.1524" layer="91"/>
-<pinref part="U$1" gate="G$1" pin="SDA"/>
-<pinref part="U1" gate="A" pin="SDA/SDI/SDIO"/>
-<wire x1="50.8" y1="5.08" x2="76.2" y2="5.08" width="0.1524" layer="91"/>
-<junction x="50.8" y="5.08"/>
-</segment>
-<segment>
-<wire x1="15.24" y1="0" x2="40.64" y2="0" width="0.1524" layer="91"/>
+<net name="N$5" class="0">
+<segment>
 <pinref part="R1" gate="G$1" pin="2"/>
 <wire x1="40.64" y1="-5.08" x2="40.64" y2="0" width="0.1524" layer="91"/>
+<pinref part="U1" gate="A" pin="SCL/SCLK"/>
+<wire x1="40.64" y1="0" x2="40.64" y2="10.16" width="0.1524" layer="91"/>
+<wire x1="40.64" y1="10.16" x2="40.64" y2="17.78" width="0.1524" layer="91"/>
+<wire x1="76.2" y1="10.16" x2="40.64" y2="10.16" width="0.1524" layer="91"/>
+<junction x="40.64" y="10.16"/>
 <pinref part="U$1" gate="G$1" pin="SCL"/>
-<wire x1="40.64" y1="0" x2="40.64" y2="10.16" width="0.1524" layer="91"/>
+<wire x1="15.24" y1="0" x2="40.64" y2="0" width="0.1524" layer="91"/>
 <junction x="40.64" y="0"/>
-<pinref part="U1" gate="A" pin="SCL/SCLK"/>
-<wire x1="40.64" y1="10.16" x2="76.2" y2="10.16" width="0.1524" layer="91"/>
+</segment>
+</net>
+<net name="N$2" class="0">
+<segment>
+<pinref part="R2" gate="G$1" pin="2"/>
+<wire x1="50.8" y1="-2.54" x2="50.8" y2="2.54" width="0.1524" layer="91"/>
+<wire x1="50.8" y1="2.54" x2="50.8" y2="7.62" width="0.1524" layer="91"/>
+<wire x1="50.8" y1="7.62" x2="50.8" y2="20.32" width="0.1524" layer="91"/>
+<pinref part="U1" gate="A" pin="SDA/SDI/SDIO"/>
+<wire x1="76.2" y1="5.08" x2="55.88" y2="5.08" width="0.1524" layer="91"/>
+<wire x1="55.88" y1="5.08" x2="55.88" y2="7.62" width="0.1524" layer="91"/>
+<wire x1="55.88" y1="7.62" x2="50.8" y2="7.62" width="0.1524" layer="91"/>
+<junction x="50.8" y="7.62"/>
+<pinref part="U$1" gate="G$1" pin="SDA"/>
+<wire x1="15.24" y1="5.08" x2="45.72" y2="5.08" width="0.1524" layer="91"/>
+<wire x1="45.72" y1="5.08" x2="45.72" y2="2.54" width="0.1524" layer="91"/>
+<wire x1="45.72" y1="2.54" x2="50.8" y2="2.54" width="0.1524" layer="91"/>
+<junction x="50.8" y="2.54"/>
+</segment>
+</net>
+<net name="N$8" class="0">
+<segment>
+<pinref part="U1" gate="A" pin="INT2"/>
+<pinref part="X1" gate="-8" pin="S"/>
+<wire x1="132.08" y1="17.78" x2="139.7" y2="17.78" width="0.1524" layer="91"/>
+</segment>
+</net>
+<net name="N$7" class="0">
+<segment>
+<pinref part="X1" gate="-2" pin="S"/>
+<pinref part="R2" gate="G$1" pin="1"/>
+<wire x1="50.8" y1="-17.78" x2="50.8" y2="-12.7" width="0.1524" layer="91"/>
 </segment>
 </net>
 <net name="N$3" class="0">
 <segment>
+<pinref part="U1" gate="A" pin="INT1"/>
+<pinref part="X1" gate="-6" pin="S"/>
+<wire x1="132.08" y1="20.32" x2="139.7" y2="20.32" width="0.1524" layer="91"/>
+</segment>
+</net>
+<net name="N$4" class="0">
+<segment>
+<pinref part="X1" gate="-4" pin="S"/>
 <pinref part="R1" gate="G$1" pin="1"/>
 <wire x1="40.64" y1="-17.78" x2="40.64" y2="-15.24" width="0.1524" layer="91"/>
-<pinref part="X3" gate="-6" pin="S"/>
-</segment>
-</net>
-<net name="N$4" class="0">
-<segment>
-<pinref part="R2" gate="G$1" pin="1"/>
-<wire x1="50.8" y1="-15.24" x2="50.8" y2="-12.7" width="0.1524" layer="91"/>
-<pinref part="X3" gate="-4" pin="S"/>
-</segment>
-</net>
+</segment>
+</net>
