File: schematics/i2c-devices.brd (EAGLE design)
At the start: 45 x 45 mm, 39 parts, among them U1 ADXL375BCCZ, U2 AD5241BRU1M-REEL7AD5241BRZ1M

Commit message: Платы, правки, накопленные изменения
Parts:
- added R7: (no value), resistor:R0805
Connections:
- net N$15: now also R7.1
- net VCC3.3: now also R7.2
Routing:
- net GND: track 28.1 -> 33.7 mm
- net N$15: track 5.47 -> 9.33 mm
Changed lines of the file:
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@@
 <layer number="37" name="tTest" color="7" fill="1" visible="no" active="yes"/>
 <layer number="38" name="bTest" color="7" fill="1" visible="no" active="yes"/>
-<layer number="39" name="tKeepout" color="4" fill="11" visible="no" active="yes"/>
+<layer number="39" name="tKeepout" color="4" fill="11" visible="yes" active="yes"/>
 <layer number="40" name="bKeepout" color="1" fill="11" visible="no" active="yes"/>
-<layer number="41" name="tRestrict" color="4" fill="10" visible="no" active="yes"/>
+<layer number="41" name="tRestrict" color="4" fill="10" visible="yes" active="yes"/>
 <layer number="42" name="bRestrict" color="1" fill="10" visible="no" active="yes"/>
 <layer number="43" name="vRestrict" color="2" fill="10" visible="no" active="yes"/>
@@
 <wire x1="45" y1="45" x2="45" y2="0" width="0.254" layer="20"/>
 <wire x1="45" y1="0" x2="0" y2="0" width="0.254" layer="20"/>
+<wire x1="21" y1="26.5" x2="24" y2="26.5" width="0.4064" layer="41"/>
+<wire x1="25" y1="16.5" x2="25" y2="23.5" width="0.254" layer="41"/>
 </plain>
 <attributes>
@@
 <element name="U$3" library="elements" package="SOIC-16" value="MC74HC4051AMC74HC4051AG" x="33" y="37" rot="R270"/>
 <element name="U$4" library="elements" package="SOIC-16" value="MC74HC4051AMC74HC4051AG" x="33" y="24" rot="R270"/>
+<element name="R7" library="resistor" package="R0805" value="" x="13" y="23" rot="R270"/>
 </elements>
 <signals>
@@
 <contactref element="C1" pad="1"/>
 <contactref element="C3" pad="C"/>
-<wire x1="21.86" y1="25.4" x2="22.86" y2="25.4" width="0.3048" layer="1"/>
 <wire x1="23.5809" y1="19.96" x2="23.5809" y2="19.16" width="0.4064" layer="1"/>
 <wire x1="22.86" y1="25.4" x2="22.86" y2="26.05" width="0.4064" layer="1"/>
 <wire x1="23.5809" y1="19.96" x2="23.6209" y2="20" width="0.4064" layer="1"/>
-<wire x1="23.6209" y1="20" x2="25.5" y2="20" width="0.4064" layer="1"/>
-<wire x1="25.5" y1="20" x2="25.5" y2="17.5" width="0.4064" layer="1"/>
-<wire x1="25.5" y1="17.5" x2="25.44" y2="17.56" width="0.4064" layer="1"/>
-<wire x1="25.44" y1="17.56" x2="23.5809" y2="17.56" width="0.4064" layer="1"/>
 <via x="27" y="32" extent="1-16" drill="1" shape="square"/>
 <wire x1="27.1953" y1="23.145" x2="29.5" y2="23.145" width="0.6096" layer="16"/>
@@
 <contactref element="U$4" pad="7"/>
 <contactref element="U$4" pad="8"/>
+<wire x1="21.86" y1="25.4" x2="21.86" y2="27.86" width="0.4064" layer="1"/>
+<wire x1="21.86" y1="27.86" x2="22" y2="28" width="0.4064" layer="1"/>
+<wire x1="22.86" y1="26.05" x2="22.86" y2="27.86" width="0.4064" layer="1"/>
+<wire x1="22.86" y1="27.86" x2="23" y2="28" width="0.4064" layer="1"/>
+<wire x1="23.6209" y1="20" x2="26.5" y2="20" width="0.4064" layer="1"/>
+<wire x1="26.5" y1="20" x2="26.5" y2="17.56" width="0.4064" layer="1"/>
+<wire x1="26.5" y1="17.56" x2="23.5809" y2="17.56" width="0.4064" layer="1"/>
 </signal>
 <signal name="N$15">
@@
 <wire x1="15.45" y1="25.36" x2="15.49" y2="25.4" width="0.4064" layer="1"/>
 <wire x1="15.49" y1="25.4" x2="20.86" y2="25.4" width="0.4064" layer="1"/>
+<contactref element="R7" pad="1"/>
+<wire x1="15.45" y1="25.36" x2="13" y2="25.36" width="0.6096" layer="1"/>
+<wire x1="13" y1="25.36" x2="13" y2="23.95" width="0.6096" layer="1"/>
 </signal>
 <signal name="N$16">
@@
 <wire x1="22.86" y1="23" x2="22.86" y2="24.75" width="0.4064" layer="1"/>
 <wire x1="23.5" y1="16.76" x2="23.5" y2="15.5" width="0.4064" layer="1"/>
-<wire x1="23.5" y1="15.5" x2="26" y2="15.5" width="0.6096" layer="1"/>
-<wire x1="26" y1="15.5" x2="26" y2="11.5" width="0.6096" layer="1"/>
+<wire x1="23.5" y1="15.5" x2="26" y2="15.5" width="0.4064" layer="1"/>
+<wire x1="26" y1="15.5" x2="26" y2="11.5" width="0.4064" layer="1"/>
 <wire x1="13.5" y1="22" x2="22.21" y2="22" width="0.6096" layer="1"/>
 <wire x1="20.8391" y1="17.5" x2="20" y2="17.5" width="0.4064" layer="1"/>
 <wire x1="20" y1="17.5" x2="19" y2="16.5" width="0.4064" layer="1"/>
-<wire x1="19" y1="16.5" x2="19" y2="11.5" width="0.6096" layer="1"/>
+<wire x1="19" y1="16.5" x2="19" y2="11.5" width="0.4064" layer="1"/>
 <wire x1="9.4792" y1="35.3986" x2="9.4792" y2="34.5" width="0.6096" layer="16"/>
 <wire x1="9.4792" y1="34.5" x2="9.4792" y2="32.5208" width="0.6096" layer="16"/>
@@
 <wire x1="19" y1="11.5" x2="17.5" y2="11.5" width="0.6096" layer="1"/>
 <wire x1="17.5" y1="11.5" x2="17.5" y2="3" width="0.6096" layer="1"/>
+<contactref element="R7" pad="2"/>
+<wire x1="13.5" y1="22" x2="13" y2="22.05" width="0" layer="19" extent="1-1"/>
 </signal>
 <signal name="SDA3.3">
@@
 <wire x1="19.5" y1="26.5" x2="20.86" y2="26.5" width="0.4064" layer="1"/>
 <wire x1="20.86" y1="26.5" x2="20.86" y2="26.05" width="0.4064" layer="1"/>
-<wire x1="24" y1="13.5" x2="22.21" y2="13.5" width="0.6096" layer="1"/>
-<wire x1="22.21" y1="13.5" x2="22.21" y2="15" width="0.6096" layer="1"/>
+<wire x1="24" y1="13.5" x2="22.21" y2="13.5" width="0.4064" layer="1"/>
+<wire x1="22.21" y1="13.5" x2="22.21" y2="15" width="0.4064" layer="1"/>
 </signal>
 <signal name="N$1">
