File: schematics/spi-devices.brd (EAGLE design)
At the start: 45 x 45 mm, 13 parts, among them J1 DM3AT-SF-PEJM5, X1 87758-1016, X2 87758-0216

Commit message: Платы, правки, накопленные изменения
Parts:
- removed R2, R4, R8: 0.75, SparkFun-Resistors:0805
- removed X1: 87758-1016, con-molex:87758-1016
- removed X2: 87758-0216, con-molex:87758-0216
- added CS_GPS, CS_SD, GND, GND8, MISO, MOSI, SCK, VCC, VCC1: (no value), wirepad:2,54/0,9
- added R1, R10, R11, R9: 0.75, SparkFun-Resistors:0805
- moved R5 31.1 mm to (12.0, 16.5), turned to 270 degrees
- moved U$1 30.8 mm to (21.7, 37.9), turned to 90 degrees
- moved R6 30.6 mm to (3.25, 18.5), turned to 90 degrees
- moved R3 28.6 mm to (5.75, 16.8), turned to 270 degrees
- moved R7 27.9 mm to (9.75, 16.5)
- moved J1 27.2 mm to (5.25, 12.5), flipped to the top
- moved C3 24.8 mm to (32.2, 11.7), flipped to the bottom, turned to 90 degrees
- moved C1 20.1 mm to (35.8, 12.5), flipped to the bottom, turned to 90 degrees
Connections:
- net N$1 renamed RF
- removed net 3.3V: C1.2, C3.A, J1.4, R2.1, U$1.1, U$1.8, U$1.9, X2.1
- removed net N$12: J1.5, R3.2, R6.1, U$1.6
- removed net N$14: J1.2, R5.2, R8.1, U$1.3
- removed net N$16: J1.3, R4.2, R7.1, U$1.26
- removed net N$2: U$1.23, X1.2
- removed net N$3: R2.2, U$1.7, X1.7
- removed net N$4: J1.7, U$1.25, X1.10
- removed net N$5: R4.1, X1.5
- removed net N$6: R5.1, X1.3
- removed net N$7: J1.6, R6.2, R7.2, R8.2
- removed net N$8: R3.1, X1.1
- new net CS_GPS: CS_GPS.1, R10.2
- new net CS_GPS_3.3: R10.1, R11.1, U$1.3
- new net CS_SD: CS_SD.1, R9.2
- new net CS_SD_3.3: J1.2, R1.1, R9.1
- new net MISO: J1.7, MISO.1, U$1.25
- new net MOSI: MOSI.1, R3.2
- new net MOSI3.3: J1.3, R3.1, R6.1, U$1.26
- new net SCK: R5.2, SCK.1
- new net SCK3.3: J1.5, R5.1, R7.1, U$1.6
- new net VCC: C1.2, C3.A, J1.4, U$1.1, U$1.23, U$1.8, U$1.9, VCC.1, VCC1.1
- net GND: now also GND.1, GND8.1, J1.6, R1.2, R11.2, R6.2, R7.2; no longer X2.2
Routing:
- net 3.3V: track 121.0 -> 0.00 mm, vias 3 -> 0
- net GND: track 140.0 -> 26.8 mm, vias 6 -> 10
- net VCC: track 0.00 -> 95.2 mm
- net N$16: track 90.4 -> 0.00 mm, vias 4 -> 0
- net N$14: track 75.6 -> 0.00 mm, vias 5 -> 0
- net SCK3.3: track 0.00 -> 72.7 mm, vias 0 -> 2
- net MISO: track 0.00 -> 62.3 mm, vias 0 -> 2
- net N$3: track 52.7 -> 0.00 mm, vias 3 -> 0
- net N$4: track 47.1 -> 0.00 mm, vias 3 -> 0
- net N$12: track 45.7 -> 0.00 mm, vias 1 -> 0
- net MOSI3.3: track 0.00 -> 34.4 mm, vias 0 -> 2
- net MOSI: track 0.00 -> 34.0 mm
- net N$7: track 33.4 -> 0.00 mm, vias 3 -> 0
- net CS_GPS_3.3: track 0.00 -> 31.0 mm, vias 0 -> 1
- net SCK: track 0.00 -> 29.6 mm
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