File: schematics/peregigateli.sch (EAGLE design)
At the start: 18 parts

Commit message: плата с пережигателями
Parts:
- added VCC3, VCC4, VCC5: LSP10, solpad:LSP10
Connections:
- new net N$10: LSP2.MP, VCC.MP
- new net N$11: R2.2, U$2Q2.G, VCC4.MP
- new net N$12: R3.2, U$3Q2.G, VCC5.MP
- net N$2: now also VCC3.MP; no longer LSP2.MP, VCC.MP
- net N$5: no longer R2.2, U$2Q2.G
- net N$8: no longer R3.2, U$3Q2.G
Changed lines of the file:
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@@
 <part name="LSP5" library="solpad" deviceset="LSP10" device=""/>
 <part name="LSP6" library="solpad" deviceset="LSP10" device=""/>
+<part name="VCC3" library="solpad" deviceset="LSP10" device=""/>
+<part name="VCC4" library="solpad" deviceset="LSP10" device=""/>
+<part name="VCC5" library="solpad" deviceset="LSP10" device=""/>
 </parts>
 <sheets>
@@
 <instance part="LSP5" gate="1" x="116.84" y="55.88"/>
 <instance part="LSP6" gate="1" x="116.84" y="66.04" rot="R180"/>
+<instance part="VCC3" gate="1" x="12.7" y="38.1" rot="R90"/>
+<instance part="VCC4" gate="1" x="53.34" y="38.1" rot="R90"/>
+<instance part="VCC5" gate="1" x="101.6" y="38.1" rot="R90"/>
 </instances>
 <busses>
@@
 <net name="N$2" class="0">
 <segment>
-<pinref part="LSP2" gate="1" pin="MP"/>
-<wire x1="27.94" y1="68.58" x2="27.94" y2="76.2" width="0.1524" layer="91"/>
-<wire x1="27.94" y1="76.2" x2="22.86" y2="76.2" width="0.1524" layer="91"/>
-<wire x1="22.86" y1="76.2" x2="22.86" y2="78.74" width="0.1524" layer="91"/>
-<pinref part="VCC" gate="1" pin="MP"/>
-<wire x1="22.86" y1="76.2" x2="15.24" y2="76.2" width="0.1524" layer="91"/>
-<wire x1="15.24" y1="76.2" x2="15.24" y2="38.1" width="0.1524" layer="91"/>
-<junction x="22.86" y="76.2"/>
 <pinref part="U$1" gate="Q2" pin="G"/>
 <wire x1="15.24" y1="38.1" x2="22.86" y2="38.1" width="0.1524" layer="91"/>
 <wire x1="15.24" y1="38.1" x2="15.24" y2="35.56" width="0.1524" layer="91"/>
+<pinref part="R1" gate="G$1" pin="2"/>
+<pinref part="VCC3" gate="1" pin="MP"/>
 <junction x="15.24" y="38.1"/>
-<pinref part="R1" gate="G$1" pin="2"/>
 </segment>
 </net>
@@
 <wire x1="63.5" y1="76.2" x2="63.5" y2="78.74" width="0.1524" layer="91"/>
 <pinref part="VCC1" gate="1" pin="MP"/>
-<wire x1="63.5" y1="76.2" x2="55.88" y2="76.2" width="0.1524" layer="91"/>
-<wire x1="55.88" y1="76.2" x2="55.88" y2="38.1" width="0.1524" layer="91"/>
-<junction x="63.5" y="76.2"/>
-<pinref part="U$2" gate="Q2" pin="G"/>
-<wire x1="55.88" y1="38.1" x2="63.5" y2="38.1" width="0.1524" layer="91"/>
-<wire x1="55.88" y1="38.1" x2="55.88" y2="35.56" width="0.1524" layer="91"/>
-<junction x="55.88" y="38.1"/>
-<pinref part="R2" gate="G$1" pin="2"/>
 </segment>
 </net>
@@
 <wire x1="111.76" y1="76.2" x2="111.76" y2="78.74" width="0.1524" layer="91"/>
 <pinref part="VCC2" gate="1" pin="MP"/>
-<wire x1="111.76" y1="76.2" x2="104.14" y2="76.2" width="0.1524" layer="91"/>
-<wire x1="104.14" y1="76.2" x2="104.14" y2="38.1" width="0.1524" layer="91"/>
-<junction x="111.76" y="76.2"/>
-<pinref part="U$3" gate="Q2" pin="G"/>
-<wire x1="104.14" y1="38.1" x2="111.76" y2="38.1" width="0.1524" layer="91"/>
-<wire x1="104.14" y1="38.1" x2="104.14" y2="35.56" width="0.1524" layer="91"/>
-<junction x="104.14" y="38.1"/>
-<pinref part="R3" gate="G$1" pin="2"/>
 </segment>
 </net>
@@
 </segment>
 </net>
+<net name="N$10" class="0">
+<segment>
+<pinref part="VCC" gate="1" pin="MP"/>
+<wire x1="22.86" y1="76.2" x2="22.86" y2="78.74" width="0.1524" layer="91"/>
+<wire x1="27.94" y1="76.2" x2="22.86" y2="76.2" width="0.1524" layer="91"/>
+<pinref part="LSP2" gate="1" pin="MP"/>
+<wire x1="27.94" y1="68.58" x2="27.94" y2="76.2" width="0.1524" layer="91"/>
+</segment>
+</net>
+<net name="N$11" class="0">
+<segment>
+<pinref part="U$2" gate="Q2" pin="G"/>
+<wire x1="55.88" y1="38.1" x2="63.5" y2="38.1" width="0.1524" layer="91"/>
+<wire x1="55.88" y1="38.1" x2="55.88" y2="35.56" width="0.1524" layer="91"/>
+<pinref part="R2" gate="G$1" pin="2"/>
+<pinref part="VCC4" gate="1" pin="MP"/>
+<junction x="55.88" y="38.1"/>
+</segment>
+</net>
+<net name="N$12" class="0">
+<segment>
+<pinref part="U$3" gate="Q2" pin="G"/>
+<wire x1="104.14" y1="38.1" x2="111.76" y2="38.1" width="0.1524" layer="91"/>
+<wire x1="104.14" y1="38.1" x2="104.14" y2="35.56" width="0.1524" layer="91"/>
+<pinref part="R3" gate="G$1" pin="2"/>
+<pinref part="VCC5" gate="1" pin="MP"/>
+<junction x="104.14" y="38.1"/>
+</segment>
+</net>
